Commit message: Refactored for headless setup

File: src/vhit_robot_moveit_config/config/vhit_robotics_rev_1.ros2_control.xacro (robot description, xacro)
@@ -1,11 +1,22 @@
 <?xml version="1.0"?>
 <robot xmlns:xacro="http://www.ros.org/wiki/xacro">
-    <xacro:macro name="vhit_robotics_rev_1_ros2_control" params="name initial_positions_file">
-        <xacro:property name="initial_positions" value="${load_yaml(initial_positions_file)['initial_positions']}"/>
+    <xacro:macro name="vhit_robotics_rev_1_ros2_control" params="name initial_positions_file hardware">
+        <xacro:property name="initial_positions" value="${xacro.load_yaml(initial_positions_file)['initial_positions']}"/>
         <ros2_control name="${name}" type="system">
-            <hardware>
-                <!-- By default, set up controllers for simulation. This won't work on real hardware -->
-                <plugin>mock_components/GenericSystem</plugin>
-            </hardware>
+            <xacro:if value="${hardware == 'mock'}">
+                <hardware>
+                    <plugin>mock_components/GenericSystem</plugin>
+                </hardware>
+            </xacro:if>
+            <xacro:if value="${hardware == 'gazebo'}">
+                <hardware>
+                    <plugin>gz_ros2_control/GazeboSimSystem</plugin>
+                </hardware>
+            </xacro:if>
+            <xacro:if value="${hardware == 'real'}">
+                <hardware>
+                    <plugin>vhit_hw/VHitSystem</plugin>
+                </hardware>
+            </xacro:if>
             <joint name="rotbase">
                 <command_interface name="position"/>

File: src/vhit_robot_moveit_config/config/vhit_robotics_rev_1.urdf.xacro (robot description, xacro)
@@ -2,8 +2,15 @@
 <robot xmlns:xacro="http://www.ros.org/wiki/xacro" name="vhit_robotics_rev_1">
     <xacro:arg name="initial_positions_file" default="initial_positions.yaml" />
+    <xacro:arg name="hardware" default="mock" />
     <!-- Import vhit_robotics_rev_1 urdf file -->
     <xacro:include filename="$(find vhit_robot_demo)/urdf/vhit_robotics_rev_1.urdf" />
     <!-- Import control_xacro -->
     <xacro:include filename="vhit_robotics_rev_1.ros2_control.xacro" />
-    <xacro:vhit_robotics_rev_1_ros2_control name="FakeSystem" initial_positions_file="$(arg initial_positions_file)"/>
+    <!-- Import gazebo_xacro -->
+    <xacro:include filename="vhit_robotics_rev_1.gazebo.xacro" />
+    <xacro:vhit_robotics_rev_1_ros2_control
+        name="FakeSystem"
+        initial_positions_file="$(arg initial_positions_file)"
+        hardware="$(arg hardware)" />
+    <xacro:vhit_robotics_rev_1_gazebo hardware="$(arg hardware)" />
 </robot>

Commit message: Fixed snap for shared memory access

File: src/vhit_robot_moveit_config/config/vhit_robotics_rev_1.ros2_control.xacro (robot description, xacro)
@@ -1,6 +1,7 @@
 <?xml version="1.0"?>
 <robot xmlns:xacro="http://www.ros.org/wiki/xacro">
-    <xacro:macro name="vhit_robotics_rev_1_ros2_control" params="name initial_positions_file hardware">
+    <xacro:macro name="vhit_robotics_rev_1_ros2_control" params="name initial_positions_file hardware elac_mapping_file">
         <xacro:property name="initial_positions" value="${xacro.load_yaml(initial_positions_file)['initial_positions']}"/>
+        <xacro:property name="elac_mapping" value="${xacro.load_yaml(elac_mapping_file)['elac_mapping']}"/>
         <ros2_control name="${name}" type="system">
             <xacro:if value="${hardware == 'mock'}">
@@ -25,5 +26,5 @@
                   <param name="initial_value">${initial_positions['rotbase']}</param>
                 </state_interface>
-                <state_interface name="velocity"/>
+                <!-- <state_interface name="velocity"/> -->
             </joint>
             <joint name="shoulder_joint">
@@ -33,5 +34,5 @@
                   <param name="initial_value">${initial_positions['shoulder_joint']}</param>
                 </state_interface>
-                <state_interface name="velocity"/>
+                <!-- <state_interface name="velocity"/> -->
             </joint>
             <joint name="elbow">
@@ -41,5 +42,5 @@
                   <param name="initial_value">${initial_positions['elbow']}</param>
                 </state_interface>
-                <state_interface name="velocity"/>
+                <!-- <state_interface name="velocity"/> -->
             </joint>
             <joint name="wrist_pitch">
@@ -49,5 +50,5 @@
                   <param name="initial_value">${initial_positions['wrist_pitch']}</param>
                 </state_interface>
-                <state_interface name="velocity"/>
+                <!-- <state_interface name="velocity"/> -->
             </joint>
             <joint name="wrist_roll">
@@ -57,5 +58,5 @@
                   <param name="initial_value">${initial_positions['wrist_roll']}</param>
                 </state_interface>
-                <state_interface name="velocity"/>
+                <!-- <state_interface name="velocity"/> -->
             </joint>
         </ros2_control>

File: src/vhit_robot_moveit_config/config/vhit_robotics_rev_1.urdf.xacro (robot description, xacro)
@@ -12,5 +12,6 @@
         name="FakeSystem"
         initial_positions_file="$(arg initial_positions_file)"
-        hardware="$(arg hardware)" />
+        hardware="$(arg hardware)"
+        elac_mapping_file="$(arg elac_mapping_file)" />
     <xacro:vhit_robotics_rev_1_gazebo hardware="$(arg hardware)" />
 </robot>
